File: schematic/UI-Micro-SD.sch (KiCad schematic (older format))
At the start: 31 parts, among them IC1 TCA9554APWR, J1 Conn_02x08_Odd_Even, J2 Conn_02x08_Odd_Even, J6 Conn_01x08, J8 Solder-Jumper-3-3-3-Open, Q1 BSS138, U1 SFV14R-3STBE1HLF, U2 DizzyBITLogo, U3 DizzyBIT-Layout

Commit message: Major Update. Changed pin configuration and board outline.
Parts:
- removed FID1, FID2: FIDUCIAL-1.5mm, fab:FIDUCIAL-1.5mm, symbol pcb:FIDUCIAL-1.5mm
- removed J6: Conn_01x08, Connector_PinHeader_2.54mm:PinHeader_1x08_P2.54mm_Vertical, symbol Connector_Generic:Conn_01x08
- removed J8: Solder-Jumper-3-3-3-Open, DizzyBit:DizzyBit-SolderJumper-3-3-3-Open, symbol DizzyBIT:Solder-Jumper-3-3-3-Open
- removed JP1: SolderJumper_2_Bridged, DizzyBit:DizzyBit-SolderJumper-2-Open, symbol Jumper:SolderJumper_2_Bridged
- removed JP3: SolderJumper_3_Bridged12, DizzyBit:DizzyBit-SolderJumper-3-Open, symbol Jumper:SolderJumper_3_Bridged12
- removed JP5: Conn_02x03_Odd_Even, DizzyBit:DizzyBit-SolderJumper-3-3-Open, symbol Connector_Generic:Conn_02x03_Odd_Even
- added J3: Conn_01x13, Connector_PinSocket_2.00mm:PinSocket_1x13_P2.00mm_Horizontal, symbol Connector_Generic:Conn_01x13
- added J4, J5, J6, JP6: Conn_01x03, Connector_PinHeader_2.00mm:PinHeader_1x03_P2.00mm_Vertical, symbol Connector_Generic:Conn_01x03
- added JP1: Conn_01x02, Connector_PinHeader_2.00mm:PinHeader_2x01_P2.00mm_Vertical, symbol Connector_Generic:Conn_01x02
- added JP5: Conn_02x04_Odd_Even, Connector_PinHeader_2.00mm:PinHeader_2x04_P2.00mm_Vertical, symbol Connector_Generic:Conn_02x04_Odd_Even
- J1, J2: footprint Connector_PinHeader_2.54mm:PinHeader_2x08_P2.54mm_Vertical -> Connector_PinSocket_2.54mm:PinSocket_2x08_P2.54mm_Vertical
- JP2: renamed from JP4; footprint DizzyBit:DizzyBit-SolderJumper-4-4-Open -> Connector_PinHeader_2.00mm:PinHeader_2x04_P2.00mm_Vertical
- JP4: renamed from JP2; footprint DizzyBit:DizzyBit-SolderJumper-5-5-Open -> Connector_PinHeader_2.00mm:PinHeader_2x05_P2.00mm_Vertical
- renumbered R5 to R4, R6 to R5, R4 to R6
Connections:
- net VBAT is gone; now on net IO26: J1.12 (Pin_12)
- net +3V3: now also J1.15 (Pin_15), J2.16 (Pin_16), J3.1 (Pin_1), J4.1 (Pin_1), J5.1 (Pin_1), J6.1 (Pin_1), JP6.1 (Pin_1); no longer J1.14 (Pin_14), J2.13 (Pin_13)
- net A0: now also J4.2 (Pin_2)
- net A1: now also J5.2 (Pin_2)
- net A2: now also J6.2 (Pin_2)
- net EN: now also J1.13 (Pin_13); no longer J2.16 (Pin_16)
- net EXT_5V: now also J2.14 (Pin_14); no longer J1.15 (Pin_15)
- net GND: now also J3.2 (Pin_2), J4.3 (Pin_3), J5.3 (Pin_3), J6.3 (Pin_3)
- net HSPI_CLK: now also J1.10 (Pin_10), JP1.1 (Pin_1); no longer J1.7 (Pin_7)
- net HSPI_MISO: now also J1.7 (Pin_7); no longer J1.13 (Pin_13)
- net HSPI_MOSI: now also J1.8 (Pin_8); no longer J1.9 (Pin_9)
- net I2C_SCL: now also J2.6 (Pin_6); no longer J2.2 (Pin_2)
- net I34: now also J2.2 (Pin_2), J3.5 (Pin_5), JP5.5 (Pin_5); no longer J1.4 (Pin_4)
- net I36: now also J1.1 (Pin_1), J3.3 (Pin_3), JP5.3 (Pin_3); no longer J1.2 (Pin_2)
- net I39: now also J1.2 (Pin_2), JP5.1 (Pin_1); no longer J1.1 (Pin_1)
- net INT: now also JP5.2 (Pin_2), JP5.4 (Pin_4), JP5.6 (Pin_6), JP5.8 (Pin_8)
- net IO1: now also J2.4 (Pin_4); no longer J2.3 (Pin_3)
- net IO15: now also J1.9 (Pin_9); no longer J1.11 (Pin_11)
- net IO16: now also J1.4 (Pin_4); no longer J2.10 (Pin_10)
- net IO17: now also J1.3 (Pin_3); no longer J2.9 (Pin_9)
- net IO2: now also J2.13 (Pin_13), JP6.3 (Pin_3); no longer J2.14 (Pin_14)
- net IO25: now also J1.6 (Pin_6); no longer J1.8 (Pin_8)
- net IO26: no longer J1.5 (Pin_5)
- net IO27: now also J1.14 (Pin_14); no longer J1.10 (Pin_10)
- net IO3: now also J2.3 (Pin_3); no longer J2.4 (Pin_4)
- net IO32: now also J1.11 (Pin_11); no longer J1.6 (Pin_6)
- net IO33: now also J1.5 (Pin_5); no longer J1.3 (Pin_3)
- net IO5: now also J2.10 (Pin_10); no longer J2.8 (Pin_8)
- net LCD_BACKLIGHT: now also JP6.2 (Pin_2)
- net P0: now also J3.13 (Pin_13)
- net P1: now also J3.12 (Pin_12)
- net P2: now also J3.11 (Pin_11)
- net P3: now also J3.10 (Pin_10)
- net P4: now also J3.9 (Pin_9)
- net P5: now also J3.8 (Pin_8)
- net P6: now also J3.7 (Pin_7)
- net P7: now also J3.6 (Pin_6)
- net VSPI_CLK: now also J2.9 (Pin_9); no longer J2.7 (Pin_7)
- net VSPI_MISO: now also J2.8 (Pin_8); no longer J2.6 (Pin_6)
- net VSPI_MOSI: now also J2.7 (Pin_7); no longer J2.1 (Pin_1)
- net at DS1.2 (A): now also JP1.2 (Pin_2)
- new net I35: J2.1 (Pin_1), J3.4 (Pin_4), JP5.7 (Pin_7)
Other:
- moved on the sheet: C1, C2, C3, DS1, IC1, JP2, JP4, Q1, R1, R2, R3, R4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
